File: mini launchpad.kicad_sch (KiCad schematic)
At the start: 145 parts, among them J1 Conn_01x08_Socket, J2 Conn_01x06_Socket, J3 Conn_01x02_Pin, J4 AudioJack3_Ground, J5 USB_C_Receptacle_USB2.0_16P, Q1 AO3401A, SW65 SW_DPDT_x2, SW66 RotaryEncoder_Switch_MP, SW67 RotaryEncoder_Switch_MP, SW68 RotaryEncoder_Switch_MP, SW69 RotaryEncoder_Switch_MP, SW70 RotaryEncoder_Switch_MP, SW71 RotaryEncoder_Switch_MP, SW72 RotaryEncoder_Switch_MP, SW73 RotaryEncoder_Switch_MP, SW75 SW_Push, SW76 SW_Push, SW77 SW_Push, SW78 SW_Push, SW79 SW_Push, SW80 SW_Push, SW81 SW_Push, SW83 SW_Push, U1 MCP23017_ML, U10 W25Q128JVS, U11 MCP23017_ML, U12 LM386, U13 LM386, U2 MCP23017_ML, U3 MCP23017_ML, U4 MCP23017_ML, U5 CP2615-xx-xM, U6 TMUX1574PW, U7 CH334R, U8 RP2040, U9 NCP1117-3.3_TO252, Y1 12MHz

Commit message: pcb update
Parts:
- removed U12, U13: LM386, Package_DIP:DIP-8_W7.62mm_Socket, symbol Amplifier_Audio:LM386
- added U14, U15: LM386, Package_SO:SOIC-8_3.9x4.9mm_P1.27mm, symbol Amplifier_Audio:LM386
- D1, D2, D3: LCSC Part (none) -> C3646935
- J1: LCSC part (none) -> C492407
- J2: LCSC Part (none) -> C5383115
- J3: LCSC Part (none) -> C42431827
- J4: LCSC Part (none) -> C4992816
- J5: footprint Connector_USB:USB_C_Receptacle_Amphenol_124019772112A -> Connector_USB:USB_C_Receptacle_G-Switch_GT-USB-7010ASV; LCSC Part (none) -> C2988369
- Q1: LCSC Part (none) -> C15127
- RV2: LCSC Part (none) -> C470285
- SW65: LCSC Part (none) -> C3664594
- SW66, SW67, SW68, SW69, SW70, SW71, SW72, SW73: LCSC Part (none) -> C202365
- U1, U11, U2, U3, U4: LCSC Part (none) -> C639770
- U10: LCSC Part (none) -> C97521
- U5: LCSC Part (none) -> C1521596
- U6: LCSC Part (none) -> C2673443
- U7: LCSC Part (none) -> C4154405
- U8: LCSC Part (none) -> C2040
- U9: LCSC Part (none) -> C154606
- Y1: LCSC C9002 -> (none); LCSC Part (none) -> C9002
Connections:
- net GND: now also U14.2 (-), U14.4 (GND), U15.2 (-), U15.4 (GND)
- net VBUS: now also U14.6 (V+), U15.6 (V+)
- net lineL: now also U15.3 (+)
- net lineR: now also U14.3 (+)
- net at C17.1: now also U15.1 (GAIN)
- net at C19.1, C20.1: now also U15.5
- net at C18.2: now also U15.7 (BYPASS)
- net at RV2.2: now also U15.8 (GAIN)
- net at C22.2: now also U14.7 (BYPASS)
- net at C23.1, C24.1: now also U14.5
- net at C21.1: now also U14.1 (GAIN)
- net at RV2.5: now also U14.8 (GAIN)

Commit message: pcb update
Parts:
- added H1, H2, H3, H4: MountingHole_Pad, MountingHole:MountingHole_3.2mm_M3_Pad_TopOnly, symbol Mechanical:MountingHole_Pad
- C1, C17, C18, C2, C21, C22: LCSC Part (none) -> C15850
- C10, C11, C12, C13, C14, C4, C5, C7, C8, C9: LCSC Part (none) -> C476766
- C15, C16: LCSC C1555 -> C1804
- C19: footprint Capacitor_SMD:C_0805_2012Metric -> Capacitor_SMD:C_1206_3216Metric
- C20, C23: value 0.05µF -> 50nF; LCSC Part (none) -> C107154
- C24: footprint Capacitor_SMD:C_0805_2012Metric -> Capacitor_SMD:C_1206_3216Metric; LCSC Part (none) -> C412252
- C3, C6: LCSC Part (none) -> C28323
- R1, R16: LCSC Part (none) -> C105872
- R10, R13: LCSC Part (none) -> C138066
- R14, R15: LCSC Part (none) -> C106232
- R2, R3: LCSC Part (none) -> C138021
- R5: LCSC Part (none) -> C11702
- R6, R8, R9: LCSC Part (none) -> C112291
- SW65: LCSC Part C3664594 -> C2848873
Connections:
- net GND: now also H1.1, H2.1, H3.1, H4.1
Other:
- note added: "mounting"

Commit message: pcb update
Connections:
- net at SW6.2: now also U1.19 (GPA2); no longer U1.2 (GPB5)
- net at SW47.2: now also U3.3 (GPB6); no longer U3.18 (GPA1)
- net at SW40.2: now also U3.17 (GPA0); no longer U3.4 (GPB7)
- net at SW23.2: now also U2.18 (GPA1); no longer U2.3 (GPB6)
- net at SW62.2: now also U4.2 (GPB5); no longer U4.19 (GPA2)
- net at U3.1 (GPB4): now also SW45.2; no longer SW37.2
- net at SW48.2: now also U3.4 (GPB7); no longer U3.17 (GPA0)
- net at U3.19 (GPA2): now also SW38.2; no longer SW46.2
- net at U3.2 (GPB5): now also SW46.2; no longer SW38.2
- net at U3.20 (GPA3): now also SW37.2; no longer SW45.2
- net at U3.21 (GPA4): now also SW36.2; no longer SW44.2
- net at U3.22 (GPA5): now also SW35.2; no longer SW43.2
- net at U3.23 (GPA6): now also SW34.2; no longer SW42.2
- net at U3.24 (GPA7): now also SW33.2; no longer SW41.2
- net at U3.25 (GPB0): now also SW41.2; no longer SW33.2
- net at U3.26 (GPB1): now also SW42.2; no longer SW34.2
- net at U3.27 (GPB2): now also SW43.2; no longer SW35.2
- net at U3.28 (GPB3): now also SW44.2; no longer SW36.2
- net at SW39.2: now also U3.18 (GPA1); no longer U3.3 (GPB6)
- net at SW69.A: now also U11.20 (GPA3); no longer U11.1 (GPB4)
- net at SW69.B: now also U11.28 (GPB3); no longer U11.21 (GPA4)
- net at SW16.2: now also U1.4 (GPB7); no longer U1.17 (GPA0)
- net at SW29.2: now also U2.1 (GPB4); no longer U2.20 (GPA3)
- net at SW18.2: now also U2.23 (GPA6); no longer U2.26 (GPB1)
- net at SW49.2: now also U4.24 (GPA7); no longer U4.25 (GPB0)
- net at SW52.2: now also U4.21 (GPA4); no longer U4.28 (GPB3)
- net at SW55.2: now also U4.18 (GPA1); no longer U4.3 (GPB6)
- net at SW22.2: now also U2.19 (GPA2); no longer U2.2 (GPB5)
- net at SW21.2: now also U2.20 (GPA3); no longer U2.1 (GPB4)
- net at U2.17 (GPA0): now also SW24.2; no longer SW32.2
- net at SW31.2: now also U2.3 (GPB6); no longer U2.18 (GPA1)
- net at SW30.2: now also U2.2 (GPB5); no longer U2.19 (GPA2)
- net at U2.21 (GPA4): now also SW20.2; no longer SW28.2
- net at U2.22 (GPA5): now also SW19.2; no longer SW27.2
- net at SW26.2: now also U2.26 (GPB1); no longer U2.23 (GPA6)
- net at U2.24 (GPA7): now also SW17.2; no longer SW25.2
- net at U2.25 (GPB0): now also SW25.2; no longer SW17.2
- net at U2.27 (GPB2): now also SW27.2; no longer SW19.2
- net at U2.28 (GPB3): now also SW28.2; no longer SW20.2
- net at U2.4 (GPB7): now also SW32.2; no longer SW24.2
- net at SW60.2: now also U4.28 (GPB3); no longer U4.21 (GPA4)
- net at SW70.A: now also U11.21 (GPA4); no longer U11.28 (GPB3)
- net at SW70.B: now also U11.1 (GPB4); no longer U11.20 (GPA3)
- net at U4.1 (GPB4): now also SW61.2; no longer SW53.2
- net at U4.17 (GPA0): now also SW56.2; no longer SW64.2
- net at SW63.2: now also U4.3 (GPB6); no longer U4.18 (GPA1)
- net at SW54.2: now also U4.19 (GPA2); no longer U4.2 (GPB5)
- net at U4.20 (GPA3): now also SW53.2; no longer SW61.2
- net at U4.22 (GPA5): now also SW51.2; no longer SW59.2
- net at U4.23 (GPA6): now also SW50.2; no longer SW58.2
- net at SW57.2: now also U4.25 (GPB0); no longer U4.24 (GPA7)
- net at U4.26 (GPB1): now also SW58.2; no longer SW50.2
- net at U4.27 (GPB2): now also SW59.2; no longer SW51.2
- net at U4.4 (GPB7): now also SW64.2; no longer SW56.2
- net at SW73.A: now also U11.24 (GPA7); no longer U11.25 (GPB0)
- net at SW73.B: now also U11.4 (GPB7); no longer U11.17 (GPA0)
- net at SW8.2: now also U1.17 (GPA0); no longer U1.4 (GPB7)
- net at SW71.A: now also U11.22 (GPA5); no longer U11.27 (GPB2)
- net at SW71.B: now also U11.2 (GPB5); no longer U11.19 (GPA2)
- net at SW12.2: now also U1.28 (GPB3); no longer U1.21 (GPA4)
- net at SW14.2: now also U1.2 (GPB5); no longer U1.19 (GPA2)
- net at SW13.2: now also U1.1 (GPB4); no longer U1.20 (GPA3)
- net at SW68.A: now also U11.19 (GPA2); no longer U11.2 (GPB5)
- net at SW68.B: now also U11.27 (GPB2); no longer U11.22 (GPA5)
- net at SW7.2: now also U1.18 (GPA1); no longer U1.3 (GPB6)
- net at SW1.2: now also U1.24 (GPA7); no longer U1.25 (GPB0)
- net at SW15.2: now also U1.3 (GPB6); no longer U1.18 (GPA1)
- net at SW10.2: now also U1.26 (GPB1); no longer U1.23 (GPA6)
- net at SW3.2: now also U1.22 (GPA5); no longer U1.27 (GPB2)
- net at U11.18 (GPA1): now also SW67.A; no longer SW72.B
- net at U11.23 (GPA6): now also SW72.A; no longer SW67.B
- net at SW66.B: now also U11.25 (GPB0); no longer U11.24 (GPA7)
- net at U11.26 (GPB1): now also SW67.B; no longer SW72.A
- net at U11.3 (GPB6): now also SW72.B; no longer SW67.A
- net at SW66.A: now also U11.17 (GPA0); no longer U11.4 (GPB7)
- net at SW4.2: now also U1.21 (GPA4); no longer U1.28 (GPB3)
- net at SW2.2: now also U1.23 (GPA6); no longer U1.26 (GPB1)
- net at SW11.2: now also U1.27 (GPB2); no longer U1.22 (GPA5)
- net at SW5.2: now also U1.20 (GPA3); no longer U1.1 (GPB4)
- net at SW9.2: now also U1.25 (GPB0); no longer U1.24 (GPA7)
Other:
- moved on the sheet: U11, U3, U4

Commit message: pcb update
Parts:
- C19: LCSC Part (none) -> C412252
- D1, D2, D3: footprint LED_SMD:LED_1206_3216Metric -> LED_THT:LED_D3.0mm; LCSC Part C3646935 -> C3028820
Changed lines of the file:
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@@
 			)
 		)
-		(property "Footprint" "LED_SMD:LED_1206_3216Metric"
+		(property "Footprint" "LED_THT:LED_D3.0mm"
 			(at 58.42 50.8 0)
 			(effects
@@
 			)
 		)
-		(property "LCSC Part" "C3646935"
+		(property "LCSC Part" "C3028820"
 			(at 58.42 50.8 90)
 			(effects
@@
 			)
 		)
-		(property "LCSC Part" ""
+		(property "LCSC Part" "C412252"
 			(at 55.88 95.25 0)
 			(effects
@@
 			)
 		)
-		(property "Footprint" "LED_SMD:LED_1206_3216Metric"
+		(property "Footprint" "LED_THT:LED_D3.0mm"
 			(at 67.31 50.8 0)
 			(effects
@@
 			)
 		)
-		(property "LCSC Part" "C3646935"
+		(property "LCSC Part" "C3028820"
 			(at 67.31 50.8 90)
 			(effects
@@
 			)
 		)
-		(property "Footprint" "LED_SMD:LED_1206_3216Metric"
+		(property "Footprint" "LED_THT:LED_D3.0mm"
 			(at 49.53 50.8 0)
 			(effects
@@
 			)
 		)
-		(property "LCSC Part" "C3646935"
+		(property "LCSC Part" "C3028820"
 			(at 49.53 50.8 90)
 			(effects

Commit message: this time I swear it's the final pcb update
Parts:
- removed SW83: SW_Push, Button_Switch_Keyboard:SW_Cherry_MX_1.00u_PCB, symbol Switch:SW_Push
Connections:
- net GPIO19: no longer names the net of U8.30 (GPIO19)
Changed lines of the file:
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@@
 		)
 	)
-	(global_label "GPIO19"
-		(shape input)
-		(at 167.64 92.71 0)
-		(fields_autoplaced yes)
-		(effects
-			(font
-				(size 1.27 1.27)
-			)
-			(justify left)
-		)
-		(property "Intersheetrefs" "${INTERSHEET_REFS}"
-			(at 177.5195 92.71 0)
-			(effects
-				(font
-					(size 1.27 1.27)
-				)
-				(justify left)
-				(hide yes)
-			)
-		)
-	)
 	(global_label "GPIO17"
 		(shape input)
@@
 		)
 	)
-	(global_label "GPIO19"
-		(shape input)
-		(at 68.58 30.48 270)
-		(fields_autoplaced yes)
-		(effects
-			(font
-				(size 1.27 1.27)
-			)
-			(justify right)
-		)
-		(property "Intersheetrefs" "${INTERSHEET_REFS}"
-			(at 68.58 40.3595 90)
-			(effects
-				(font
-					(size 1.27 1.27)
-				)
-				(justify right)
-				(hide yes)
-			)
-		)
-	)
 	(global_label "GPIO20"
 		(shape input)
@@
 	(symbol
 		(lib_id "power:GND")
-		(at 68.58 20.32 180)
-		(unit 1)
-		(exclude_from_sim no)
-		(in_bom yes)
-		(on_board yes)
-		(dnp no)
-		(fields_autoplaced yes)
-		(property "Reference" "#PWR0159"
-			(at 68.58 13.97 0)
-			(effects
-				(font
-					(size 1.27 1.27)
-				)
-				(hide yes)
-			)
-		)
-		(property "Value" "GND"
-			(at 68.58 15.24 0)
-			(effects
-				(font
-					(size 1.27 1.27)
-				)
-			)
-		)
-		(property "Footprint" ""
-			(at 68.58 20.32 0)
-			(effects
-				(font
-					(size 1.27 1.27)
-				)
-				(hide yes)
-			)
-		)
-		(property "Datasheet" ""
-			(at 68.58 20.32 0)
-			(effects
-				(font
-					(size 1.27 1.27)
-				)
-				(hide yes)
-			)
-		)
-		(property "Description" "Power symbol creates a global label with name \"GND\" , ground"
-			(at 68.58 20.32 0)
-			(effects
-				(font
-					(size 1.27 1.27)
-				)
-				(hide yes)
-			)
-		)
-		(pin "1"
-		)
-		(instances
-			(project "mini launchpad"
-				(path "/53b873fe-fce8-4274-bbb6-cd8ec25e3130"
-					(reference "#PWR0159")
-					(unit 1)
-				)
-			)
-		)
-	)
-	(symbol
-		(lib_id "power:GND")
 		(at 101.6 97.79 0)
 		(unit 1)
@@
 					(unit 1)
 				)
-			)
-		)
-	)
-	(symbol
-		(lib_id "Switch:SW_Push")
-		(at 68.58 25.4 270)
-		(unit 1)
-		(exclude_from_sim no)
-		(in_bom yes)
-		(on_board yes)
-		(dnp no)
-		(property "Reference" "SW83"
-			(at 69.342 21.59 90)
-			(effects
-				(font
-					(size 1.27 1.27)
-				)
-				(justify left)
-			)
-		)
-		(property "Value" "SW_Push"
-			(at 67.31 24.1301 90)
-			(effects
-				(font
-					(size 1.27 1.27)
-				)
-				(justify right)
-				(hide yes)
-			)
-		)
-		(property "Footprint" "Button_Switch_Keyboard:SW_Cherry_MX_1.00u_PCB"
-			(at 73.66 25.4 0)
-			(effects
-				(font
-					(size 1.27 1.27)
-				)
-				(hide yes)
-			)
-		)
-		(property "Datasheet" "~"
-			(at 73.66 25.4 0)
-			(effects
-				(font
-					(size 1.27 1.27)
-				)
-				(hide yes)
-			)
-		)
-		(property "Description" "Push button switch, generic, two pins"
-			(at 68.58 25.4 0)
-			(effects
-				(font
-					(size 1.27 1.27)
-				)
-				(hide yes)
-			)
-		)
-		(pin "2"
-		)
-		(pin "1"
-		)
-		(instances
-			(project "mini launchpad"
-				(path "/53b873fe-fce8-4274-bbb6-cd8ec25e3130"
-					(reference "SW83")
-					(unit 1)
-				)
