File: mini launchpad.kicad_pcb (KiCad board)
At the start: 2 copper layers, 69 parts, among them U1 MCP23017_ML, U2 MCP23017_ML, U3 MCP23017_ML, U4 MCP23017_ML

Commit message: pcb update
Parts:
- removed A2: RaspberryPi_Pico, Module:RaspberryPi_Pico_Common_THT
- added C1: 10µF, Capacitor_SMD:C_0201_0603Metric, F.Cu at (138.5, 122.1)
- added C10: 100nF, Capacitor_SMD:C_0201_0603Metric, F.Cu at (140.9, 129.1)
- added C11: 100nF, Capacitor_SMD:C_0201_0603Metric, F.Cu at (143.4, 122.1)
- added C12: 100nF, Capacitor_SMD:C_0201_0603Metric, F.Cu at (143.4, 123.9)
- added C13: 100nF, Capacitor_SMD:C_0201_0603Metric, F.Cu at (143.4, 125.6)
- added C14: 100nF, Capacitor_SMD:C_0201_0603Metric, F.Cu at (143.4, 127.4)
- added C15: 22pF, Capacitor_SMD:C_0402_1005Metric, F.Cu at (138.7, 135.5)
- added C16: 22pF, Capacitor_SMD:C_0402_1005Metric, F.Cu at (138.7, 137.5)
- added C2: 10µF, Capacitor_SMD:C_0201_0603Metric, F.Cu at (138.5, 123.9)
- added C3: 1µF, Capacitor_SMD:C_0201_0603Metric, F.Cu at (138.5, 125.6)
- added C4: 100nF, Capacitor_SMD:C_0201_0603Metric, F.Cu at (138.5, 127.4)
- added C5: 100nF, Capacitor_SMD:C_0201_0603Metric, F.Cu at (138.5, 129.1)
- added C6: 1µF, Capacitor_SMD:C_0201_0603Metric, F.Cu at (140.9, 122.1)
- added C7: 100nF, Capacitor_SMD:C_0201_0603Metric, F.Cu at (140.9, 123.9)
- added C8: 100nF, Capacitor_SMD:C_0201_0603Metric, F.Cu at (140.9, 125.6)
- added C9: 100nF, Capacitor_SMD:C_0201_0603Metric, F.Cu at (140.9, 127.4)
- added JP1: Jumper_2_Open, Jumper:Jumper_Harwin_S1621_P10.9mm, F.Cu at (144.7, 71.9)
- added P1: USB_C_Plug_USB2.0, Connector_USB:USB_C_Plug_JAE_DX07P024AJ1, F.Cu at (142.3, 97.1)
- added R1: 5.1K, Resistor_SMD:R_0402_1005Metric, F.Cu at (138.7, 83.2)
- added R2: 27, Resistor_SMD:R_0402_1005Metric, F.Cu at (138.7, 85.2)
- added R3: 27, Resistor_SMD:R_0402_1005Metric, F.Cu at (138.7, 87.2)
- added R4: 10K, Resistor_SMD:R_0402_1005Metric, F.Cu at (138.7, 89.2)
- added R5: 1K, Resistor_SMD:R_0402_1005Metric, F.Cu at (138.7, 91.2)
- added R7: 1k, Resistor_SMD:R_0402_1005Metric, F.Cu at (138.7, 93.2)
- added SW65: SW_DPDT_x2, Button_Switch_THT:SW_E-Switch_EG2219_DPDT_Angled, F.Cu at (141.1, 55.4)
- added U10: W25Q128JVS, Package_SO:SOIC-8_5.3x5.3mm_P1.27mm, F.Cu at (145.3, 85.7)
- added U5: CP2615-xx-xM, Package_DFN_QFN:QFN-32-1EP_5x5mm_P0.5mm_EP3.3x3.3mm, F.Cu at (148.3, 124.9)
- added U6: TMUX1574PW, Package_SO:TSSOP-16_4.4x5mm_P0.65mm, F.Cu at (142.0, 118.0)
- added U7: CH334R, Connector_USB:USB_C_Plug_Molex_105444, F.Cu at (142.1, 102.9)
- added U8: RP2040, Package_DFN_QFN:QFN-56-1EP_7x7mm_P0.4mm_EP3.2x3.2mm, F.Cu at (141.9, 110.0)
- added U9: NCP1117-3.3_TO252, Package_TO_SOT_SMD:TO-252-2, F.Cu at (144.2, 78.2)
- added Y1: 12MHz, Crystal:Crystal_SMD_3225-4Pin_3.2x2.5mm, F.Cu at (139.9, 132.3)
- moved U1 72.8 mm to (141.4, 22.9)
- moved U2 72.8 mm to (141.4, 31.2)
- moved U3 72.8 mm to (141.4, 39.5)
- moved U4 72.8 mm to (141.4, 47.7)
- moved SW17 2.42 mm to (56.8, 21.3)
- moved SW18 2.42 mm to (56.8, 36.4)
- moved SW19 2.42 mm to (56.8, 51.5)
- moved SW20 2.42 mm to (56.8, 66.6)
- moved SW21 2.42 mm to (56.8, 81.7)
- moved SW22 2.42 mm to (56.8, 96.7)
- moved SW23 2.42 mm to (56.8, 111.8)
- moved SW24 2.42 mm to (56.8, 126.9)
- moved SW25 2.42 mm to (71.9, 21.3)
- moved SW26 2.42 mm to (71.9, 36.4)
- moved SW27 2.42 mm to (71.9, 51.5)
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Connections:
- U1 pad 16: unconnected-(U1-INTA-Pad16) -> INT1
- U2 pad 16: unconnected-(U2-INTA-Pad16) -> INT2
- U3 pad 16: unconnected-(U3-INTA-Pad16) -> INT3
- U4 pad 16: unconnected-(U4-INTA-Pad16) -> INT4
Other:
- board outline added: 8.2 x 5 mm

Commit message: pcb update
Parts:
- added D1: LED, LED_SMD:LED_1206_3216Metric, F.Cu at (210.3, 85.2)
- added SW66: RotaryEncoder_Switch_MP, Rotary_Encoder:RotaryEncoder_Alps_EC11E-Switch_Vertical_H20mm_MountingHoles, F.Cu at (164.2, 34.1)
- added SW67: RotaryEncoder_Switch_MP, Rotary_Encoder:RotaryEncoder_Alps_EC11E-Switch_Vertical_H20mm_MountingHoles, F.Cu at (164.2, 49.4)
- added SW68: RotaryEncoder_Switch_MP, Rotary_Encoder:RotaryEncoder_Alps_EC11E-Switch_Vertical_H20mm_MountingHoles, F.Cu at (164.2, 64.7)
- added SW69: RotaryEncoder_Switch_MP, Rotary_Encoder:RotaryEncoder_Alps_EC11E-Switch_Vertical_H20mm_MountingHoles, F.Cu at (182.8, 34.1)
- added SW70: RotaryEncoder_Switch_MP, Rotary_Encoder:RotaryEncoder_Alps_EC11E-Switch_Vertical_H20mm_MountingHoles, F.Cu at (182.8, 49.4)
- added SW71: RotaryEncoder_Switch_MP, Rotary_Encoder:RotaryEncoder_Alps_EC11E-Switch_Vertical_H20mm_MountingHoles, F.Cu at (182.8, 64.7)
- added SW72: RotaryEncoder_Switch_MP, Rotary_Encoder:RotaryEncoder_Alps_EC11E-Switch_Vertical_H20mm_MountingHoles, F.Cu at (201.3, 34.1)
- added SW73: RotaryEncoder_Switch_MP, Rotary_Encoder:RotaryEncoder_Alps_EC11E-Switch_Vertical_H20mm_MountingHoles, F.Cu at (201.3, 49.4)
- added SW74: SW_Push, Button_Switch_Keyboard:SW_Cherry_MX_1.00u_PCB, F.Cu at (172.3, 77.2)
- added SW75: SW_Push, Button_Switch_Keyboard:SW_Cherry_MX_1.00u_PCB, F.Cu at (172.3, 92.3)
- added SW76: SW_Push, Button_Switch_Keyboard:SW_Cherry_MX_1.00u_PCB, F.Cu at (172.3, 107.4)
- added SW77: SW_Push, Button_Switch_Keyboard:SW_Cherry_MX_1.00u_PCB, F.Cu at (187.4, 77.2)
- added SW78: SW_Push, Button_Switch_Keyboard:SW_Cherry_MX_1.00u_PCB, F.Cu at (187.4, 92.3)
- added SW79: SW_Push, Button_Switch_Keyboard:SW_Cherry_MX_1.00u_PCB, F.Cu at (187.4, 107.4)
- added SW80: SW_Push, Button_Switch_Keyboard:SW_Cherry_MX_1.00u_PCB, F.Cu at (202.5, 77.2)
- added SW81: SW_Push, Button_Switch_Keyboard:SW_Cherry_MX_1.00u_PCB, F.Cu at (202.5, 92.3)
- added SW82: SW_Push, Button_Switch_Keyboard:SW_Cherry_MX_1.00u_PCB, F.Cu at (202.5, 107.4)
- added SW84: RotaryEncoder_Switch_MP, Rotary_Encoder:RotaryEncoder_Alps_EC11E-Switch_Vertical_H20mm_MountingHoles, F.Cu at (201.3, 64.7)
- added U11: MCP23017_ML, Package_DFN_QFN:QFN-28-1EP_6x6mm_P0.65mm_EP4.25x4.25mm, F.Cu at (211.6, 78.9)
Connections:
- R5 pad 2: Net-(JP1-A) -> Net-(R5-Pad2)
- U6 pad 10: unconnected-(U6-S3B-Pad10) -> PI_BLCK
- U6 pad 13: unconnected-(U6-S4B-Pad13) -> PI_LRCLK
- U6 pad 6: unconnected-(U6-S2B-Pad6) -> PI_DIN
- U8 pad 38: unconnected-(U8-GPIO26_ADC0-Pad38) -> PI_BLCK
- U8 pad 39: unconnected-(U8-GPIO27_ADC1-Pad39) -> PI_LRCLK
- U8 pad 40: unconnected-(U8-GPIO28_ADC2-Pad40) -> PI_DIN
- U8 pad 8: unconnected-(U8-GPIO6-Pad8) -> INT5
- U8 pad 9: unconnected-(U8-GPIO7-Pad9) -> INT5

Commit message: pcb update
Parts:
- removed JP1: Jumper_2_Open, Jumper:Jumper_Harwin_S1621_P10.9mm
- removed SW84: RotaryEncoder_Switch_MP, Rotary_Encoder:RotaryEncoder_Alps_EC11E-Switch_Vertical_H20mm_MountingHoles
- added C17: 10µF, Capacitor_SMD:C_0201_0603Metric, F.Cu at (181.0, 140.0)
- added C18: 10µF, Capacitor_SMD:C_0201_0603Metric, F.Cu at (181.0, 141.8)
- added C19: 250µF, Capacitor_SMD:C_0201_0603Metric, F.Cu at (181.0, 143.5)
- added C20: 0.05µF, Capacitor_SMD:C_0201_0603Metric, F.Cu at (181.0, 145.3)
- added C21: 10µF, Capacitor_SMD:C_0201_0603Metric, F.Cu at (183.4, 136.5)
- added C22: 10µF, Capacitor_SMD:C_0201_0603Metric, F.Cu at (183.4, 138.3)
- added C23: 0.05µF, Capacitor_SMD:C_0201_0603Metric, F.Cu at (183.4, 140.0)
- added C24: 250µF, Capacitor_SMD:C_0201_0603Metric, F.Cu at (183.4, 141.8)
- added D2: LED, LED_SMD:LED_1206_3216Metric, F.Cu at (168.9, 159.5)
- added D3: LED, LED_SMD:LED_1206_3216Metric, F.Cu at (168.9, 162.9)
- added R10: 10, Resistor_SMD:R_0402_1005Metric, F.Cu at (170.5, 142.6)
- added R11: 10K, Resistor_SMD:R_0402_1005Metric, F.Cu at (170.5, 144.6)
- added R12: 10K, Resistor_SMD:R_0402_1005Metric, F.Cu at (170.5, 146.6)
- added R13: 10, Resistor_SMD:R_0402_1005Metric, F.Cu at (173.4, 136.6)
- added R14: 220, Resistor_SMD:R_0402_1005Metric, F.Cu at (173.4, 138.6)
- added R15: 220, Resistor_SMD:R_0402_1005Metric, F.Cu at (173.4, 140.6)
- added R6: 220, Resistor_SMD:R_0402_1005Metric, F.Cu at (167.6, 146.6)
- added R8: 220, Resistor_SMD:R_0402_1005Metric, F.Cu at (170.5, 138.6)
- added R9: 220, Resistor_SMD:R_0402_1005Metric, F.Cu at (170.5, 140.6)
- added RV2: R_Potentiometer_Dual, Potentiometer_THT:Potentiometer_Alpha_RD902F-40-00D_Dual_Vertical, F.Cu at (153.0, 140.0)
- added SW83: SW_Push, Button_Switch_Keyboard:SW_Cherry_MX_1.00u_PCB, F.Cu at (143.8, 65.9)
- added U12: LM386, Package_DIP:DIP-8_W7.62mm_Socket, F.Cu at (159.1, 96.5)
- added U13: LM386, Package_DIP:DIP-8_W7.62mm_Socket, F.Cu at (170.8, 96.5)
- moved SW49 121.5 mm to (98.5, 141.3)
- moved SW50 121.5 mm to (98.5, 156.4)
- moved SW9 120.1 mm to (38.2, 141.3)
- moved SW10 120.1 mm to (38.2, 156.4)
- moved SW31 91.9 mm to (83.4, 20.6)
- moved SW32 91.9 mm to (83.4, 35.7)
- moved SW57 91.8 mm to (113.6, 111.2)
- moved SW58 91.8 mm to (113.6, 126.2)
- moved SW59 91.8 mm to (113.6, 141.3)
- moved SW60 91.8 mm to (113.6, 156.4)
- moved SW17 89.9 mm to (53.3, 111.2)
- moved SW19 89.9 mm to (53.3, 141.3)
- moved SW18 89.9 mm to (53.3, 126.2)
- moved SW20 89.9 mm to (53.3, 156.4)
- moved D1 82.1 mm to (168.9, 156.1)
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Connections:
- D1 pad 1: unconnected-(D1-K-Pad1) -> GND
- D1 pad 2: unconnected-(D1-A-Pad2) -> Net-(D1-A)
- SW75 pad 2: unconnected-(SW75-Pad2) -> GPIO24
- SW76 pad 2: unconnected-(SW76-Pad2) -> GPIO23
- SW77 pad 2: unconnected-(SW77-Pad2) -> GPIO22
- SW78 pad 2: unconnected-(SW78-Pad2) -> GPIO21
- SW79 pad 2: unconnected-(SW79-Pad2) -> GPIO20
- SW80 pad 2: unconnected-(SW80-Pad2) -> GPIO18
- SW81 pad 2: unconnected-(SW81-Pad2) -> GPIO17
- SW82 pad 2: unconnected-(SW82-Pad2) -> GPIO16
- U8 pad 16: unconnected-(U8-GPIO13-Pad16) -> GPIO13
- U8 pad 17: unconnected-(U8-GPIO14-Pad17) -> GPIO14
- U8 pad 18: unconnected-(U8-GPIO15-Pad18) -> GPIO15
- U8 pad 27: unconnected-(U8-GPIO16-Pad27) -> GPIO16
- U8 pad 28: unconnected-(U8-GPIO17-Pad28) -> GPIO17
- U8 pad 29: unconnected-(U8-GPIO18-Pad29) -> GPIO18
- U8 pad 30: unconnected-(U8-GPIO19-Pad30) -> GPIO19
- U8 pad 31: unconnected-(U8-GPIO20-Pad31) -> GPIO20
- U8 pad 32: unconnected-(U8-GPIO21-Pad32) -> GPIO21
- U8 pad 34: unconnected-(U8-GPIO22-Pad34) -> GPIO22
- U8 pad 35: unconnected-(U8-GPIO23-Pad35) -> GPIO23
- U8 pad 36: unconnected-(U8-GPIO24-Pad36) -> GPIO24

Commit message: pcb update
Parts:
- removed SW82: SW_Push, Button_Switch_Keyboard:SW_Cherry_MX_1.00u_PCB
- added J1: Conn_01x08_Socket, Connector_PinHeader_2.54mm:PinHeader_1x08_P2.54mm_Vertical, F.Cu at (312.7, 96.7)
- added J2: Conn_01x06_Socket, Connector_PinHeader_2.54mm:PinHeader_1x06_P2.54mm_Vertical, F.Cu at (304.4, 139.9)
- added Q1: AO3401A, Package_TO_SOT_SMD:SOT-23, F.Cu at (324.7, 119.3)
- R14, R15: value 220 -> 100
- U7: footprint Connector_USB:USB_C_Plug_Molex_105444 -> Package_SO:QSOP-16_3.9x4.9mm_P0.635mm
- moved SW83 255.1 mm to (397.5, 39.2)
- moved SW74 254.0 mm to (382.4, 69.4)
- moved SW79 254.0 mm to (382.4, 144.8)
- moved SW80 254.0 mm to (397.5, 9.04)
- moved SW81 254.0 mm to (397.5, 24.1)
- moved SW32 168.4 mm to (101.1, 203.2)
- moved U5 163.3 mm to (318.6, 116.0)
- moved SW31 160.7 mm to (101.1, 180.3)
- moved U8 158.4 mm to (311.4, 150.5)
- moved C21 153.8 mm to (336.7, 124.7)
- moved C22 153.8 mm to (336.7, 126.5)
- moved C23 153.8 mm to (336.7, 128.2)
- moved C24 153.8 mm to (336.7, 130.0)
- moved R10 153.8 mm to (323.8, 130.8)
- moved R11 153.8 mm to (323.8, 132.8)
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Connections:
- P1 pad A6: Net-(P1-D+) -> /D+
- P1 pad A7: Net-(P1-D-) -> /D-
- R2 pad 1: D+1 -> 1D+
- R3 pad 2: D-1 -> 1D-
- R6 pad 1: GPIO15 -> GPIO16
- R8 pad 1: GPIO14 -> GPIO15
- R9 pad 1: GPIO13 -> GPIO14
- SW18 pad 2: Net-(U2-GPA7) -> Net-(U2-GPB1)
- SW19 pad 2: Net-(U2-GPB1) -> Net-(U2-GPB2)
- SW20 pad 2: Net-(U2-GPA6) -> Net-(U2-GPB3)
- SW21 pad 2: Net-(U2-GPB2) -> Net-(U2-GPB4)
- SW22 pad 2: Net-(U2-GPA5) -> Net-(U2-GPB5)
- SW23 pad 2: Net-(U2-GPB3) -> Net-(U2-GPB6)
- SW24 pad 2: Net-(U2-GPA4) -> Net-(U2-GPB7)
- SW25 pad 2: Net-(U2-GPB4) -> Net-(U2-GPA7)
- SW26 pad 2: Net-(U2-GPA3) -> Net-(U2-GPA6)
- SW27 pad 2: Net-(U2-GPB5) -> Net-(U2-GPA5)
- SW28 pad 2: Net-(U2-GPA2) -> Net-(U2-GPA4)
- SW29 pad 2: Net-(U2-GPB6) -> Net-(U2-GPA3)
- SW30 pad 2: Net-(U2-GPA1) -> Net-(U2-GPA2)
- SW31 pad 2: Net-(U2-GPB7) -> Net-(U2-GPA1)
- SW34 pad 2: Net-(U3-GPA7) -> Net-(U3-GPB1)
- SW35 pad 2: Net-(U3-GPB1) -> Net-(U3-GPB2)
- SW36 pad 2: Net-(U3-GPA6) -> Net-(U3-GPB3)
- SW37 pad 2: Net-(U3-GPB2) -> Net-(U3-GPB4)
- SW38 pad 2: Net-(U3-GPA5) -> Net-(U3-GPB5)
- SW39 pad 2: Net-(U3-GPB3) -> Net-(U3-GPB6)
- SW40 pad 2: Net-(U3-GPA4) -> Net-(U3-GPB7)
- SW41 pad 2: Net-(U3-GPB4) -> Net-(U3-GPA7)
- SW42 pad 2: Net-(U3-GPA3) -> Net-(U3-GPA6)
- SW43 pad 2: Net-(U3-GPB5) -> Net-(U3-GPA5)
- SW44 pad 2: Net-(U3-GPA2) -> Net-(U3-GPA4)
- SW45 pad 2: Net-(U3-GPB6) -> Net-(U3-GPA3)
- SW46 pad 2: Net-(U3-GPA1) -> Net-(U3-GPA2)
- SW47 pad 2: Net-(U3-GPB7) -> Net-(U3-GPA1)
- SW50 pad 2: Net-(U4-GPA7) -> Net-(U4-GPB1)
- SW51 pad 2: Net-(U4-GPB1) -> Net-(U4-GPB2)
- SW52 pad 2: Net-(U4-GPA6) -> Net-(U4-GPB3)
- SW53 pad 2: Net-(U4-GPB2) -> Net-(U4-GPB4)
- SW54 pad 2: Net-(U4-GPA5) -> Net-(U4-GPB5)
- SW55 pad 2: Net-(U4-GPB3) -> Net-(U4-GPB6)
- SW56 pad 2: Net-(U4-GPA4) -> Net-(U4-GPB7)
- SW57 pad 2: Net-(U4-GPB4) -> Net-(U4-GPA7)
- SW58 pad 2: Net-(U4-GPA3) -> Net-(U4-GPA6)
- SW59 pad 2: Net-(U4-GPB5) -> Net-(U4-GPA5)
- SW60 pad 2: Net-(U4-GPA2) -> Net-(U4-GPA4)
- SW61 pad 2: Net-(U4-GPB6) -> Net-(U4-GPA3)
- SW62 pad 2: Net-(U4-GPA1) -> Net-(U4-GPA2)
- SW63 pad 2: Net-(U4-GPB7) -> Net-(U4-GPA1)
- SW66 pad A: Net-(U11-GPB0) -> Net-(U11-GPB7)
- SW66 pad B: Net-(U11-GPA0) -> Net-(U11-GPA7)
- SW67 pad A: Net-(U11-GPB1) -> Net-(U11-GPB6)
- SW67 pad B: Net-(U11-GPA1) -> Net-(U11-GPA6)
- SW68 pad A: Net-(U11-GPB2) -> Net-(U11-GPB5)
- SW68 pad B: Net-(U11-GPA2) -> Net-(U11-GPA5)
- SW69 pad A: Net-(U11-GPB3) -> Net-(U11-GPB4)
- SW69 pad B: Net-(U11-GPA3) -> Net-(U11-GPA4)
- SW70 pad A: Net-(U11-GPB7) -> Net-(U11-GPB3)
- SW70 pad B: Net-(U11-GPA7) -> Net-(U11-GPA3)
- SW71 pad A: Net-(U11-GPB6) -> Net-(U11-GPB2)
- SW71 pad B: Net-(U11-GPA6) -> Net-(U11-GPA2)
- SW72 pad A: Net-(U11-GPB5) -> Net-(U11-GPB1)
- SW72 pad B: Net-(U11-GPA5) -> Net-(U11-GPA1)
- SW73 pad A: Net-(U11-GPB4) -> Net-(U11-GPB0)
- SW73 pad B: Net-(U11-GPA4) -> Net-(U11-GPA0)
- U5 pad 4: D+2 -> 2D+
- U5 pad 5: D-2 -> 2D-
- U6 pad 12: unconnected-(U6-D4-Pad12) -> LRCLK
- U6 pad 7: unconnected-(U6-D2-Pad7) -> DIN
- U6 pad 9: unconnected-(U6-D3-Pad9) -> BLCK
Routing:
- net SDA: track 0.00 -> 274.3 mm, vias 0 -> 5
- net SCK: track 0.00 -> 233.8 mm, vias 0 -> 5
- net Net-(U11-GPA7): track 0.00 -> 90.4 mm, vias 0 -> 1
- net Net-(U11-GPB7): track 0.00 -> 90.1 mm
- net Net-(U4-GPB0): track 0.00 -> 86.0 mm
- net Net-(U3-GPB0): track 0.00 -> 86.0 mm
- net Net-(U1-GPB0): track 0.00 -> 86.0 mm
- net Net-(U2-GPB0): track 0.00 -> 86.0 mm
- net Net-(U2-GPA7): track 0.00 -> 83.3 mm
- net Net-(U3-GPB7): track 0.00 -> 82.9 mm
- net Net-(U1-GPB7): track 0.00 -> 82.9 mm
- net Net-(U4-GPB7): track 0.00 -> 82.8 mm
- net Net-(U2-GPB7): track 0.00 -> 82.8 mm
- net Net-(U4-GPA7): track 0.00 -> 82.6 mm
- net Net-(U3-GPA7): track 0.00 -> 82.6 mm
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- added copper zone on In2.Cu, net +3V3
- added copper zone on B.Cu, net GND
Other:
- board size 8.2 x 5 mm -> 271.8 x 202.6 mm
- copper layers 2 -> 4

Commit message: pcb update
Parts:
- removed SW74: SW_Push, Button_Switch_Keyboard:SW_Cherry_MX_1.00u_PCB
- added J3: Conn_01x02_Pin, Connector_PinHeader_2.54mm:PinHeader_1x02_P2.54mm_Horizontal, F.Cu at (227.7, 75.6)
- added J4: AudioJack3_Ground, Connector_Audio:Jack_3.5mm_CUI_SJ1-3524N_Horizontal, F.Cu at (255.0, 19.8)
- C1, C10, C11, C12, C13, C14, C17, C18, C19, C2, C20, C21, C22, C23, C24, C3, C4, C5, C6, C7, C8, C9: footprint Capacitor_SMD:C_0201_0603Metric -> Capacitor_SMD:C_0805_2012Metric
- C15, C16: footprint Capacitor_SMD:C_0402_1005Metric -> Capacitor_SMD:C_0805_2012Metric
- moved SW80 207.6 mm to (212.5, 103.2)
- moved SW81 183.0 mm to (232.5, 103.2)
- moved SW83 175.0 mm to (222.5, 43.2)
- moved U6 173.5 mm to (187.5, 47.0)
- moved SW79 164.4 mm to (222.5, 183.2)
- moved U5 153.5 mm to (187.2, 36.6), turned to -90 degrees
- moved Q1 151.8 mm to (187.0, 55.4)
- moved C19 146.6 mm to (233.7, 25.1), turned to 90 degrees
- moved C13 146.0 mm to (192.8, 88.9), turned to 180 degrees
- moved C16 144.8 mm to (187.4, 84.6), turned to -90 degrees
- moved C20 143.7 mm to (235.7, 29.0), turned to 90 degrees
- moved C21 142.7 mm to (231.6, 28.2), turned to 180 degrees
- moved C5 142.6 mm to (192.8, 90.9), turned to 180 degrees
- moved C10 142.5 mm to (197.0, 83.7), turned to -90 degrees
- moved C15 142.1 mm to (190.5, 81.5)
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Connections:
- R14 pad 1: outL -> Net-(J4-PadT)
- R15 pad 1: outR -> Net-(J4-PadR)
- U8 pad 9: INT5 -> INT6
Routing:
- net INT1: track 0.00 -> 198.6 mm, vias 1 -> 2
- net INT2: track 0.00 -> 152.1 mm, vias 1 -> 2
- net INT6: track 0.70 -> 121.6 mm, vias 1 -> 2
- net INT5: track 0.00 -> 118.2 mm, vias 1 -> 2
- net lineL: track 0.00 -> 112.2 mm
- net GPIO16: track 0.00 -> 104.1 mm
- net INT3: track 0.00 -> 100.1 mm, vias 1 -> 2
- net lineR: track 0.00 -> 85.4 mm
- net Net-(U1-GPA0): track 79.1 -> 0.00 mm
- net 1D-: track 0.00 -> 74.5 mm, vias 0 -> 2
- net 1D+: track 0.00 -> 72.5 mm, vias 0 -> 2
- net GPIO23: track 0.00 -> 68.4 mm
- net GPIO22: track 0.00 -> 62.0 mm
- net INT4: track 0.00 -> 60.8 mm, vias 1 -> 2
- net SCK: track 233.8 -> 293.1 mm, vias 5 -> 6
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Other:
- board size 271.8 x 202.6 mm -> 241.2 x 202.7 mm

Commit message: pcb update
Parts:
- removed P1: USB_C_Plug_USB2.0, Connector_USB:USB_C_Plug_JAE_DX07P024AJ1
- added J5: USB_C_Receptacle_USB2.0_16P, Connector_USB:USB_C_Receptacle_Amphenol_124019772112A, F.Cu at (186.4, 16.8)
- added R16: 5.1K, Resistor_SMD:R_0402_1005Metric, F.Cu at (183.0, 22.4)
- moved R1 5.77 mm to (190.1, 22.5)
- moved C11 1.45 mm to (198.6, 97.5)
- moved C8 1.42 mm to (202.2, 97.4)
- moved C2 1.20 mm to (204.3, 45.2)
- moved J4 0.11 mm to (254.9, 19.7)
Routing:
- net GPIO20: track 0.00 -> 102.1 mm, vias 0 -> 1
- net GPIO21: track 0.00 -> 94.9 mm, vias 0 -> 1
- net GPIO14: track 0.00 -> 78.7 mm, vias 0 -> 4
- net PI_BLCK: track 0.00 -> 70.5 mm, vias 0 -> 2
- net Net-(U1-GPA0): track 0.00 -> 68.9 mm
- net PI_I²S: track 0.00 -> 67.8 mm, vias 0 -> 2
- net PI_LRCLK: track 0.00 -> 67.3 mm, vias 0 -> 2
- net GPIO19: track 0.00 -> 65.9 mm, vias 0 -> 2
- net PI_DIN: track 0.00 -> 57.9 mm, vias 0 -> 2
- net GPIO24: track 0.00 -> 45.8 mm, vias 0 -> 1
- net GPIO13: track 0.00 -> 43.5 mm
- net GPIO15: track 0.00 -> 24.6 mm, vias 0 -> 2
- net BLCK: track 0.00 -> 23.7 mm
- net DIN: track 0.00 -> 23.7 mm, vias 0 -> 1
- net LRCLK: track 0.00 -> 20.9 mm
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Other:
- board size 241.2 x 202.7 mm -> 241.2 x 180.3 mm

Commit message: pcb update
Parts:
- J5: footprint Connector_USB:USB_C_Receptacle_Amphenol_124019772112A -> Connector_USB:USB_C_Receptacle_G-Switch_GT-USB-7010ASV
- moved R16 2.18 mm to (182.0, 24.4)
- moved R1 2.10 mm to (190.3, 24.6)
- moved J5 1.24 mm to (186.3, 18.1)
- moved U7 1.10 mm to (186.5, 27.8)
Routing:
- net Net-(SW65A-B): track 30.3 -> 24.0 mm
- net /D-: track 10.1 -> 6.19 mm, vias 2 -> 0
- net Net-(J5-CC2): track 6.11 -> 3.58 mm
- net /D+: track 9.25 -> 7.11 mm, vias 2 -> 0
- net 1D-: track 74.5 -> 73.4 mm
- net 2D-: track 4.91 -> 3.78 mm
- net 2D+: track 4.86 -> 3.73 mm
- net 1D+: track 72.5 -> 71.4 mm
- net +3V3: track 94.9 -> 94.0 mm
