File: mini launchpad.kicad_pcb (KiCad board)
At the start: 4 copper layers, 241.2 x 180.3 mm, 145 parts, among them J1 Conn_01x08_Socket, J2 Conn_01x06_Socket, J3 Conn_01x02_Pin, J4 AudioJack3_Ground, J5 USB_C_Receptacle_USB2.0_16P, Q1 AO3401A, SW65 SW_DPDT_x2, SW66 RotaryEncoder_Switch_MP, SW67 RotaryEncoder_Switch_MP, SW68 RotaryEncoder_Switch_MP, SW69 RotaryEncoder_Switch_MP, SW70 RotaryEncoder_Switch_MP, SW71 RotaryEncoder_Switch_MP, SW72 RotaryEncoder_Switch_MP, SW73 RotaryEncoder_Switch_MP, SW75 SW_Push, SW76 SW_Push, SW77 SW_Push, SW78 SW_Push, SW79 SW_Push, SW80 SW_Push, SW81 SW_Push, SW83 SW_Push, U1 MCP23017_ML, U10 W25Q128JVS, U11 MCP23017_ML, U12 LM386, U13 LM386, U2 MCP23017_ML, U3 MCP23017_ML, U4 MCP23017_ML, U5 CP2615-xx-xM, U6 TMUX1574PW, U7 CH334R, U8 RP2040, U9 NCP1117-3.3_TO252, Y1 12MHz

Commit message: pcb update
Parts:
- removed U12, U13: LM386, Package_DIP:DIP-8_W7.62mm_Socket
- added H1: MountingHole_Pad, MountingHole:MountingHole_3.2mm_M3_Pad_TopOnly, F.Cu at (251.5, 185.6)
- added H2: MountingHole_Pad, MountingHole:MountingHole_3.2mm_M3_Pad_TopOnly, F.Cu at (251.5, 55.2)
- added H3: MountingHole_Pad, MountingHole:MountingHole_3.2mm_M3_Pad_TopOnly, F.Cu at (40.0, 37.0)
- added H4: MountingHole_Pad, MountingHole:MountingHole_3.2mm_M3_Pad_TopOnly, F.Cu at (40.0, 178.3)
- added U14: LM386, Package_SO:SOIC-8_3.9x4.9mm_P1.27mm, F.Cu at (243.2, 40.1)
- added U15: LM386, Package_SO:SOIC-8_3.9x4.9mm_P1.27mm, F.Cu at (242.0, 28.0)
- C19, C24: footprint Capacitor_SMD:C_0805_2012Metric -> Capacitor_SMD:C_1206_3216Metric
- C20, C23: value 0.05µF -> 50nF
- moved R11 17.9 mm to (235.1, 41.9), turned to 90 degrees
- moved C18 11.8 mm to (244.4, 23.6), turned to -90 degrees
- moved C21 11.6 mm to (237.7, 38.1)
- moved R12 2.03 mm to (238.0, 41.4), turned to 90 degrees
- moved C19 0.10 mm to (233.6, 25.1)
Routing:
- net lineL: track 112.2 -> 77.5 mm
- net lineR: track 85.4 -> 70.5 mm
- net GND: track 97.4 -> 111.9 mm, vias 29 -> 30
- net Net-(C21-Pad1): track 16.4 -> 2.08 mm, vias 1 -> 0
- net Net-(C21-Pad2): track 2.10 -> 14.2 mm
- net Net-(RV2-Pad2): track 31.7 -> 21.1 mm
- net Net-(C19-Pad1): track 7.89 -> 15.6 mm
- net VBUS: track 91.5 -> 97.7 mm, vias 0 -> 1
- net Net-(C17-Pad1): track 18.8 -> 12.7 mm, vias 1 -> 0
- net Net-(C19-Pad2): track 23.9 -> 18.8 mm
- net Net-(U14-BYPASS): track 2.33 -> 6.56 mm
- net Net-(RV2-Pad5): track 25.6 -> 22.4 mm, vias 0 -> 1
- net Net-(U15-BYPASS): track 6.66 -> 5.01 mm
- net Net-(C23-Pad1): track 14.4 -> 15.4 mm

Commit message: pcb update
Parts:
- C1, C10, C11, C12, C13, C14, C15, C16, C17, C18, C19, C2, C20, C21, C22, C23, C24, C3, C4, C5, C6, C7, C8, C9, D1, D2, D3, H1, H2, H3, H4, J1, J2, J5, Q1, R1, R10, R11, R12, R13, R14, R15, R16, R2, R3, R4, R5, R6, R7, R8, R9, U1, U10, U11, U14, U15, U2, U3, U4, U5, U6, U7, U8, U9, Y1: moved to B.Cu
- moved R15 62.4 mm to (203.4, 54.8), turned to 180 degrees
- moved C24 49.9 mm to (200.6, 53.0), turned to -90 degrees
- moved C22 46.1 mm to (197.5, 46.9), turned to 0 degrees
- moved J3 42.1 mm to (187.9, 89.4), turned to -90 degrees
- moved U14 40.7 mm to (203.1, 47.4), turned to 180 degrees
- moved H2 36.3 mm to (234.5, 23.1), turned to 180 degrees
- moved C14 35.7 mm to (187.0, 83.5), turned to 0 degrees
- moved J4 35.0 mm to (220.0, 19.7)
- moved C16 35.0 mm to (222.4, 84.6)
- moved C23 34.9 mm to (203.9, 51.5), turned to 0 degrees
- moved C18 34.6 mm to (214.3, 40.7), turned to 90 degrees
- moved R13 31.6 mm to (206.9, 51.5), turned to 0 degrees
- moved R14 31.3 mm to (219.1, 31.8)
- moved R12 30.6 mm to (208.2, 48.2), turned to 180 degrees
- moved C21 29.4 mm to (209.2, 45.4), turned to 0 degrees
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Connections:
- SW1 pad 2: Net-(U1-GPB0) -> Net-(U1-GPA7)
- SW10 pad 2: Net-(U1-GPA6) -> Net-(U1-GPB1)
- SW11 pad 2: Net-(U1-GPA5) -> Net-(U1-GPB2)
- SW12 pad 2: Net-(U1-GPA4) -> Net-(U1-GPB3)
- SW13 pad 2: Net-(U1-GPA3) -> Net-(U1-GPB4)
- SW14 pad 2: Net-(U1-GPA2) -> Net-(U1-GPB5)
- SW15 pad 2: Net-(U1-GPA1) -> Net-(U1-GPB6)
- SW16 pad 2: Net-(U1-GPA0) -> Net-(U1-GPB7)
- SW17 pad 2: Net-(U2-GPB0) -> Net-(U2-GPA7)
- SW18 pad 2: Net-(U2-GPB1) -> Net-(U2-GPA6)
- SW19 pad 2: Net-(U2-GPB2) -> Net-(U2-GPA5)
- SW2 pad 2: Net-(U1-GPB1) -> Net-(U1-GPA6)
- SW20 pad 2: Net-(U2-GPB3) -> Net-(U2-GPA4)
- SW21 pad 2: Net-(U2-GPB4) -> Net-(U2-GPA3)
- SW22 pad 2: Net-(U2-GPB5) -> Net-(U2-GPA2)
- SW23 pad 2: Net-(U2-GPB6) -> Net-(U2-GPA1)
- SW24 pad 2: Net-(U2-GPB7) -> Net-(U2-GPA0)
- SW25 pad 2: Net-(U2-GPA7) -> Net-(U2-GPB0)
- SW26 pad 2: Net-(U2-GPA6) -> Net-(U2-GPB1)
- SW27 pad 2: Net-(U2-GPA5) -> Net-(U2-GPB2)
- SW28 pad 2: Net-(U2-GPA4) -> Net-(U2-GPB3)
- SW29 pad 2: Net-(U2-GPA3) -> Net-(U2-GPB4)
- SW3 pad 2: Net-(U1-GPB2) -> Net-(U1-GPA5)
- SW30 pad 2: Net-(U2-GPA2) -> Net-(U2-GPB5)
- SW31 pad 2: Net-(U2-GPA1) -> Net-(U2-GPB6)
- SW32 pad 2: Net-(U2-GPA0) -> Net-(U2-GPB7)
- SW33 pad 2: Net-(U3-GPB0) -> Net-(U3-GPA7)
- SW34 pad 2: Net-(U3-GPB1) -> Net-(U3-GPA6)
- SW35 pad 2: Net-(U3-GPB2) -> Net-(U3-GPA5)
- SW36 pad 2: Net-(U3-GPB3) -> Net-(U3-GPA4)
- SW37 pad 2: Net-(U3-GPB4) -> Net-(U3-GPA3)
- SW38 pad 2: Net-(U3-GPB5) -> Net-(U3-GPA2)
- SW39 pad 2: Net-(U3-GPB6) -> Net-(U3-GPA1)
- SW4 pad 2: Net-(U1-GPB3) -> Net-(U1-GPA4)
- SW40 pad 2: Net-(U3-GPB7) -> Net-(U3-GPA0)
- SW41 pad 2: Net-(U3-GPA7) -> Net-(U3-GPB0)
- SW42 pad 2: Net-(U3-GPA6) -> Net-(U3-GPB1)
- SW43 pad 2: Net-(U3-GPA5) -> Net-(U3-GPB2)
- SW44 pad 2: Net-(U3-GPA4) -> Net-(U3-GPB3)
- SW45 pad 2: Net-(U3-GPA3) -> Net-(U3-GPB4)
- SW46 pad 2: Net-(U3-GPA2) -> Net-(U3-GPB5)
- SW47 pad 2: Net-(U3-GPA1) -> Net-(U3-GPB6)
- SW48 pad 2: Net-(U3-GPA0) -> Net-(U3-GPB7)
- SW49 pad 2: Net-(U4-GPB0) -> Net-(U4-GPA7)
- SW5 pad 2: Net-(U1-GPB4) -> Net-(U1-GPA3)
- SW50 pad 2: Net-(U4-GPB1) -> Net-(U4-GPA6)
- SW51 pad 2: Net-(U4-GPB2) -> Net-(U4-GPA5)
- SW52 pad 2: Net-(U4-GPB3) -> Net-(U4-GPA4)
- SW53 pad 2: Net-(U4-GPB4) -> Net-(U4-GPA3)
- SW54 pad 2: Net-(U4-GPB5) -> Net-(U4-GPA2)
- SW55 pad 2: Net-(U4-GPB6) -> Net-(U4-GPA1)
- SW56 pad 2: Net-(U4-GPB7) -> Net-(U4-GPA0)
- SW57 pad 2: Net-(U4-GPA7) -> Net-(U4-GPB0)
- SW58 pad 2: Net-(U4-GPA6) -> Net-(U4-GPB1)
- SW59 pad 2: Net-(U4-GPA5) -> Net-(U4-GPB2)
- SW6 pad 2: Net-(U1-GPB5) -> Net-(U1-GPA2)
- SW60 pad 2: Net-(U4-GPA4) -> Net-(U4-GPB3)
- SW61 pad 2: Net-(U4-GPA3) -> Net-(U4-GPB4)
- SW62 pad 2: Net-(U4-GPA2) -> Net-(U4-GPB5)
- SW63 pad 2: Net-(U4-GPA1) -> Net-(U4-GPB6)
- SW64 pad 2: Net-(U4-GPA0) -> Net-(U4-GPB7)
- SW66 pad A: Net-(U11-GPB7) -> Net-(U11-GPA0)
- SW66 pad B: Net-(U11-GPA7) -> Net-(U11-GPB0)
- SW67 pad A: Net-(U11-GPB6) -> Net-(U11-GPA1)
- SW67 pad B: Net-(U11-GPA6) -> Net-(U11-GPB1)
- SW68 pad A: Net-(U11-GPB5) -> Net-(U11-GPA2)
- SW68 pad B: Net-(U11-GPA5) -> Net-(U11-GPB2)
- SW69 pad A: Net-(U11-GPB4) -> Net-(U11-GPA3)
- SW69 pad B: Net-(U11-GPA4) -> Net-(U11-GPB3)
- SW7 pad 2: Net-(U1-GPB6) -> Net-(U1-GPA1)
- SW70 pad A: Net-(U11-GPB3) -> Net-(U11-GPA4)
- SW70 pad B: Net-(U11-GPA3) -> Net-(U11-GPB4)
- SW71 pad A: Net-(U11-GPB2) -> Net-(U11-GPA5)
- SW71 pad B: Net-(U11-GPA2) -> Net-(U11-GPB5)
- SW72 pad A: Net-(U11-GPB1) -> Net-(U11-GPA6)
- SW72 pad B: Net-(U11-GPA1) -> Net-(U11-GPB6)
- SW73 pad A: Net-(U11-GPB0) -> Net-(U11-GPA7)
- SW73 pad B: Net-(U11-GPA0) -> Net-(U11-GPB7)
- SW8 pad 2: Net-(U1-GPB7) -> Net-(U1-GPA0)
- SW9 pad 2: Net-(U1-GPA7) -> Net-(U1-GPB0)
Routing:
- net +3V3: track 94.0 -> 229.3 mm, vias 19 -> 20
- net GPIO16: track 104.1 -> 0.00 mm
- net GPIO20: track 102.1 -> 0.00 mm, vias 1 -> 0
- net GPIO21: track 94.9 -> 0.00 mm, vias 1 -> 0
- net PI_BLCK: track 70.5 -> 0.00 mm, vias 2 -> 0
- net GPIO23: track 69.8 -> 0.00 mm
- net PI_I²S: track 67.8 -> 0.00 mm, vias 2 -> 0
- net PI_LRCLK: track 67.3 -> 0.00 mm, vias 2 -> 0
- net GPIO19: track 65.9 -> 0.00 mm, vias 2 -> 0
- net GPIO22: track 62.0 -> 0.00 mm
- net PI_DIN: track 57.9 -> 0.00 mm, vias 2 -> 0
- net GPIO14: track 78.7 -> 28.6 mm, vias 4 -> 2
- net INT6: track 121.6 -> 168.7 mm, vias 2 -> 0
- net GPIO24: track 45.8 -> 0.00 mm, vias 1 -> 0
- net GPIO15: track 24.6 -> 69.6 mm, vias 2 -> 0
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- added copper zone on F.Cu, net GND
- removed copper zone on In2.Cu, net +3V3
- removed copper zone on B.Cu, net GND
Other:
- board size 241.2 x 180.3 mm -> 206.2 x 180.3 mm

Commit message: pcb update
Parts:
- D1, D2, D3: footprint LED_SMD:LED_1206_3216Metric -> LED_THT:LED_D3.0mm; moved to F.Cu
- moved H2 43.8 mm to (222.5, 65.2)
- moved Q1 21.0 mm to (191.0, 44.3), turned to -90 degrees
- moved J1 18.6 mm to (195.7, 43.2)
- moved J2 18.6 mm to (180.4, 45.7)
- moved U6 18.6 mm to (187.1, 52.7)
- moved C24 16.4 mm to (192.7, 38.6), turned to 180 degrees
- moved R15 15.8 mm to (196.7, 40.5)
- moved C2 15.1 mm to (191.9, 74.6)
- moved C1 15.1 mm to (184.1, 64.6)
- moved U9 15.1 mm to (189.1, 69.9)
- moved C21 11.6 mm to (204.8, 34.7)
- moved C22 11.6 mm to (193.1, 36.2)
- moved C23 11.6 mm to (199.4, 40.8)
- moved R12 11.6 mm to (203.8, 37.5)
- moved R13 11.6 mm to (202.5, 40.8)
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Routing:
- net +3V3: track 229.3 -> 89.8 mm, vias 20 -> 21
- net GPIO16: track 0.00 -> 116.3 mm, vias 0 -> 2
- net GPIO20: track 0.00 -> 102.2 mm, vias 0 -> 1
- net PI_I²S: track 0.00 -> 82.3 mm, vias 0 -> 2
- net GPIO21: track 0.00 -> 79.0 mm, vias 0 -> 1
- net PI_BLCK: track 0.00 -> 75.9 mm, vias 0 -> 2
- net PI_LRCLK: track 0.00 -> 67.5 mm, vias 0 -> 2
- net GPIO22: track 0.00 -> 67.0 mm, vias 0 -> 1
- net PI_DIN: track 0.00 -> 66.3 mm, vias 0 -> 2
- net GPIO23: track 0.00 -> 65.6 mm, vias 0 -> 1
- net GPIO24: track 0.00 -> 52.5 mm, vias 0 -> 1
- net GPIO19: track 0.00 -> 45.5 mm, vias 0 -> 1
- net GPIO18: track 0.00 -> 40.3 mm, vias 0 -> 1
- net lineL: track 67.5 -> 34.6 mm
- net Net-(U5-I2S_SDIN): track 56.9 -> 26.5 mm
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- added copper zone on In1.Cu, net +3V3
Other:
- board size 206.2 x 180.3 mm -> 206.5 x 180.3 mm

Commit message: this time I swear it's the final pcb update
Parts:
- removed SW83: SW_Push, Button_Switch_Keyboard:SW_Cherry_MX_1.00u_PCB
- J4, SW65: moved to B.Cu
- moved SW65 8.75 mm to (199.2, 27.2), turned to 0 degrees
- moved RV2 6.82 mm to (207.6, 50.8)
- turned J4 to 0 degrees
Connections:
- U8 pad 30: GPIO19 -> unconnected-(U8-GPIO19-Pad30)
Routing:
- net GPIO19: track 45.5 -> 0.00 mm, vias 1 -> 0
- net Net-(RV2-Pad2): track 27.7 -> 13.0 mm
- net Net-(C17-Pad2): track 29.1 -> 19.9 mm
- net Net-(J4-PadR): track 38.9 -> 31.5 mm
- net lineL: track 34.6 -> 40.4 mm
- net Net-(RV2-Pad5): track 29.0 -> 32.5 mm
- net lineR: track 29.4 -> 31.8 mm
- net Net-(C21-Pad2): track 23.5 -> 21.8 mm
- net Net-(J4-PadT): track 8.26 -> 8.99 mm
- net Net-(SW65A-B): track 23.6 -> 22.9 mm
