File: pcb/mini launchpad.kicad_pcb (KiCad board)
At the start: 4 copper layers, 206.5 x 180.3 mm, 148 parts, among them J1 Conn_01x08_Socket, J2 Conn_01x06_Socket, J3 Conn_01x02_Pin, J4 AudioJack3_Ground, J5 USB_C_Receptacle_USB2.0_16P, Q1 AO3401A, SW65 SW_DPDT_x2, SW66 RotaryEncoder_Switch_MP, SW67 RotaryEncoder_Switch_MP, SW68 RotaryEncoder_Switch_MP, SW69 RotaryEncoder_Switch_MP, SW70 RotaryEncoder_Switch_MP, SW71 RotaryEncoder_Switch_MP, SW72 RotaryEncoder_Switch_MP, SW73 RotaryEncoder_Switch_MP, SW75 SW_Push, SW76 SW_Push, SW77 SW_Push, SW78 SW_Push, SW79 SW_Push, SW80 SW_Push, SW81 SW_Push, U1 MCP23017_ML, U10 W25Q128JVS, U11 MCP23017_ML, U14 LM386, U15 LM386, U2 MCP23017_ML, U3 MCP23017_ML, U4 MCP23017_ML, U5 CP2615-xx-xM, U6 TMUX1574PW, U7 CH334R, U8 RP2040, U9 NCP1117-3.3_TO252, Y1 12MHz

Commit message: basic code
Connections:
- U11 pad 15: INT6 -> unconnected-(U11-INTB-Pad15)
- U8 pad 2: INT1 -> SDA
- U8 pad 3: INT2 -> SCK
- U8 pad 4: INT3 -> INT1
- U8 pad 5: INT4 -> INT2
- U8 pad 6: SDA -> INT3
- U8 pad 7: SCK -> INT4
- U8 pad 9: INT6 -> unconnected-(U8-GPIO7-Pad9)
Routing:
- net INT6: track 165.5 -> 0.00 mm
- net INT1: track 218.8 -> 211.5 mm
- net SDA: track 305.2 -> 299.1 mm
- net INT4: track 75.4 -> 80.0 mm
- net INT3: track 130.4 -> 133.9 mm
- net INT2: track 154.7 -> 157.5 mm
- net SCK: track 302.8 -> 301.9 mm
