File: pcb/mini launchpad.kicad_sch (KiCad schematic)
At the start: 148 parts, among them J1 Conn_01x08_Socket, J2 Conn_01x06_Socket, J3 Conn_01x02_Pin, J4 AudioJack3_Ground, J5 USB_C_Receptacle_USB2.0_16P, Q1 AO3401A, SW65 SW_DPDT_x2, SW66 RotaryEncoder_Switch_MP, SW67 RotaryEncoder_Switch_MP, SW68 RotaryEncoder_Switch_MP, SW69 RotaryEncoder_Switch_MP, SW70 RotaryEncoder_Switch_MP, SW71 RotaryEncoder_Switch_MP, SW72 RotaryEncoder_Switch_MP, SW73 RotaryEncoder_Switch_MP, SW75 SW_Push, SW76 SW_Push, SW77 SW_Push, SW78 SW_Push, SW79 SW_Push, SW80 SW_Push, SW81 SW_Push, U1 MCP23017_ML, U10 W25Q128JVS, U11 MCP23017_ML, U14 LM386, U15 LM386, U2 MCP23017_ML, U3 MCP23017_ML, U4 MCP23017_ML, U5 CP2615-xx-xM, U6 TMUX1574PW, U7 CH334R, U8 RP2040, U9 NCP1117-3.3_TO252, Y1 12MHz

Commit message: basic code
Connections:
- net INT1: now also U8.4 (GPIO2); no longer U8.2 (GPIO0)
- net INT2: now also U8.5 (GPIO3); no longer U8.3 (GPIO1)
- net INT3: now also U8.6 (GPIO4); no longer U8.4 (GPIO2)
- net INT4: now also U8.7 (GPIO5); no longer U8.5 (GPIO3)
- net SCK: now also U8.3 (GPIO1); no longer U8.7 (GPIO5)
- net SDA: now also U8.2 (GPIO0); no longer U8.6 (GPIO4)
- net INT6: no longer names the net of U8.9 (GPIO7)
- net INT6: no longer U11.15 (INTB)
Changed lines of the file:
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@@
-		)
-	)
-	(global_label "INT6"
-		(shape output)
-		(at 232.41 194.31 0)
-		(fields_autoplaced yes)
-		(effects
-			(font
-				(size 1.27 1.27)
-			)
-			(justify left)
-		)
-		(property "Intersheetrefs" "${INTERSHEET_REFS}"
-			(at 239.5076 194.31 0)
-			(effects
-				(font
-					(size 1.27 1.27)
-				)
-				(justify left)
-				(hide yes)
-			)
 		)
 	)
@@
 	(global_label "INT4"
 		(shape input)
-		(at 167.64 52.07 0)
-		(fields_autoplaced yes)
-		(effects
-			(font
-				(size 1.27 1.27)
-			)
-			(justify left)
-		)
-		(property "Intersheetrefs" "${INTERSHEET_REFS}"
-			(at 174.7376 52.07 0)
+		(at 167.64 57.15 0)
+		(fields_autoplaced yes)
+		(effects
+			(font
+				(size 1.27 1.27)
+			)
+			(justify left)
+		)
+		(property "Intersheetrefs" "${INTERSHEET_REFS}"
+			(at 174.7376 57.15 0)
 			(effects
 				(font
@@
 	(global_label "INT3"
 		(shape input)
-		(at 167.64 49.53 0)
-		(fields_autoplaced yes)
-		(effects
-			(font
-				(size 1.27 1.27)
-			)
-			(justify left)
-		)
-		(property "Intersheetrefs" "${INTERSHEET_REFS}"
-			(at 174.7376 49.53 0)
+		(at 167.64 54.61 0)
+		(fields_autoplaced yes)
+		(effects
+			(font
+				(size 1.27 1.27)
+			)
+			(justify left)
+		)
+		(property "Intersheetrefs" "${INTERSHEET_REFS}"
+			(at 174.7376 54.61 0)
 			(effects
 				(font
@@
 	(global_label "SCK"
 		(shape input)
-		(at 167.64 57.15 0)
-		(fields_autoplaced yes)
-		(effects
-			(font
-				(size 1.27 1.27)
-			)
-			(justify left)
-		)
-		(property "Intersheetrefs" "${INTERSHEET_REFS}"
-			(at 174.3747 57.15 0)
+		(at 167.64 46.99 0)
+		(fields_autoplaced yes)
+		(effects
+			(font
+				(size 1.27 1.27)
+			)
+			(justify left)
+		)
+		(property "Intersheetrefs" "${INTERSHEET_REFS}"
+			(at 174.3747 46.99 0)
 			(effects
 				(font
@@
 	(global_label "INT2"
 		(shape input)
-		(at 167.64 46.99 0)
-		(fields_autoplaced yes)
-		(effects
-			(font
-				(size 1.27 1.27)
-			)
-			(justify left)
-		)
-		(property "Intersheetrefs" "${INTERSHEET_REFS}"
-			(at 174.7376 46.99 0)
-			(effects
-				(font
-					(size 1.27 1.27)
-				)
-				(justify left)
-				(hide yes)
-			)
-		)
-	)
-	(global_label "INT6"
-		(shape input)
-		(at 167.64 62.23 0)
-		(fields_autoplaced yes)
-		(effects
-			(font
-				(size 1.27 1.27)
-			)
-			(justify left)
-		)
-		(property "Intersheetrefs" "${INTERSHEET_REFS}"
-			(at 174.7376 62.23 0)
+		(at 167.64 52.07 0)
+		(fields_autoplaced yes)
+		(effects
+			(font
+				(size 1.27 1.27)
+			)
+			(justify left)
+		)
+		(property "Intersheetrefs" "${INTERSHEET_REFS}"
+			(at 174.7376 52.07 0)
 			(effects
 				(font
@@
 	(global_label "INT1"
 		(shape input)
-		(at 167.64 44.45 0)
-		(fields_autoplaced yes)
-		(effects
-			(font
-				(size 1.27 1.27)
-			)
-			(justify left)
-		)
-		(property "Intersheetrefs" "${INTERSHEET_REFS}"
-			(at 174.7376 44.45 0)
+		(at 167.64 49.53 0)
+		(fields_autoplaced yes)
+		(effects
+			(font
+				(size 1.27 1.27)
+			)
+			(justify left)
+		)
+		(property "Intersheetrefs" "${INTERSHEET_REFS}"
+			(at 174.7376 49.53 0)
 			(effects
 				(font
@@
 	(global_label "SDA"
 		(shape bidirectional)
-		(at 167.64 54.61 0)
-		(fields_autoplaced yes)
-		(effects
-			(font
-				(size 1.27 1.27)
-			)
-			(justify left)
-		)
-		(property "Intersheetrefs" "${INTERSHEET_REFS}"
-			(at 175.3046 54.61 0)
-			(effects
-				(font
+		(at 167.64 44.45 0)
+		(fields_autoplaced yes)
+		(effects
+			(font
+				(size 1.27 1.27)
+			)
+			(justify left)
+		)
+		(property "Intersheetrefs" "${INTERSHEET_REFS}"
+			(at 175.3046 44.45 0)
+			(effects
+				(font
